Commit message: Consolidate workspace: unify controllers, fix URDF, add simulation launch
- Unified amiibot_controllers.yaml into amiibot_controller/config/ (single source of truth)
- Fixed URDF: wheel radius (0.0855), separation (0.345), left wheel axis (0,-1,0)
- Fixed IMU/laser link names in gazebo.xacro to match URDF
- Added amiibot_simulation.launch.py as simulation entry point
- Added controller.launch.py and joystick_teleop.launch.py to amiibot_controller
- Added twist_mux and joystick config files
- Fixed amiibot_base.launch.py and amiibot_base_odrive.launch.py (broken refs removed)
- EKF added to simulation launch with use_sim_time=True
- Nav2 odom_topic corrected to /odometry/filtered
- Removed legacy/duplicate files: roboclaw config, amiibot_slam2, .xacro.save

Co-Authored-By: Claude Sonnet 4.6 <noreply@anthropic.com>

File: src/amiibot_description/urdf/amiibot.urdf.xacro (robot description, xacro)
@@ -1,10 +1,11 @@
 <?xml version="1.0"?>
 <robot name="amiibot" xmlns:xacro="http://www.ros.org/wiki/xacro">
-<!--
-    <xacro:include filename="amiibot_base.xacro"/>
-    <xacro:include filename="amiibot_ros2_control.xacro"/>
+    <!-- Argument to enable simulation mode (disables real hardware) -->
+    <xacro:arg name="is_simulation" default="false"/>
+    <!-- Base model -->
+    <xacro:include filename="$(find amiibot_description)/urdf/amiibot_base.xacro"/>
+    <!-- Gazebo plugins and sensors (only for simulation) -->
     <xacro:include filename="$(find amiibot_description)/urdf/amiibot_gazebo.xacro"/>
--->
-    <xacro:include filename="$(find amiibot_description)/urdf/amiibot_base.xacro"/>
-    <xacro:include filename="$(find amiibot_description)/urdf/amiibot_ros2_control.xacro"/>
+    <!-- ROS2 Control: conditional between sim and real hardware -->
+    <xacro:include filename="$(find amiibot_description)/urdf/amiibot_ros2_control.xacro" />
 </robot>

File: src/amiibot_description/urdf/amiibot_base.xacro (robot description, xacro)
@@ -165,5 +165,5 @@
         <child link="left_wheel"/>
         <origin xyz="0 0.1725 0.0455" rpy="0 0 0"/>
-        <axis xyz="0 1 0"/>
+        <axis xyz="0 -1 0"/>
         <dynamics damping="0.2"/>
     </joint>

File: src/amiibot_description/urdf/amiibot_gazebo.xacro (robot description, xacro)
@@ -23,35 +23,22 @@
       <maxVel>0.1</maxVel>
     </gazebo>
-    <!-- ROS 2 Control -->
+    <!-- ROS 2 Control Plugin -->
     <gazebo>
-        <!-- ROS 2 Humble -->
-        <xacro:if value="$(arg is_ignition)">
-          <plugin filename="ign_ros2_control-system" name="ign_ros2_control::IgnitionROS2ControlPlugin">
-              <parameters>$(find amiibot_controller)/config/amiibot_controllers.yaml</parameters>
-          </plugin>
-          <plugin filename="ignition-gazebo-imu-system" name="ignition::gazebo::systems::Imu">
-          </plugin>
-          <plugin filename="ignition-gazebo-sensors-system" name="ignition::gazebo::systems::Sensors">
+        <plugin filename="ign_ros2_control-system" name="ign_ros2_control::IgnitionROS2ControlPlugin">
+            <parameters>$(find amiibot_controller)/config/amiibot_controllers.yaml</parameters>
+        </plugin>
+        <!-- IMU and LiDAR Sensors System -->
+        <plugin filename="ignition-gazebo-imu-system" name="ignition::gazebo::systems::Imu">
+        </plugin>
+        <plugin filename="ignition-gazebo-sensors-system" name="ignition::gazebo::systems::Sensors">
             <render_engine>ogre2</render_engine>
-          </plugin>
-        </xacro:if>
-        <!-- ROS 2 Iron or above -->
-        <xacro:unless value="$(arg is_ignition)">
-          <plugin filename="gz_ros2_control-system" name="gz_ros2_control::GazeboSimROS2ControlPlugin">
-              <parameters>$(find amiibot_controller)/config/amiibot_controllers.yaml</parameters>
-          </plugin>
-          <plugin filename="gz-sim-imu-system" name="gz::sim::systems::Imu">
-          </plugin>
-          <plugin filename="gz-sim-sensors-system" name="gz::sim::systems::Sensors">
-          <render_engine>ogre2</render_engine>
-          </plugin>
-        </xacro:unless>
+        </plugin>
     </gazebo>
   <!-- IMU -->
-  <gazebo reference="imu_link">
+  <gazebo reference="imu">
     <sensor name="imu" type="imu">
         <always_on>true</always_on>
         <update_rate>100</update_rate>
-        <gz_frame_id>imu_link</gz_frame_id>
+        <gz_frame_id>imu</gz_frame_id>
         <topic>imu</topic>
         <imu>
@@ -99,31 +86,31 @@
     </sensor>
   </gazebo>
-  <gazebo reference="laser_link">
-    <sensor name="lidar" type="gpu_ray">
-        <always_on>true</always_on>
-        <update_rate>5</update_rate>
-        <visualize>true</visualize>
-        <topic>scan</topic>
-        <gz_frame_id>laser_link</gz_frame_id>
-        <ray>
-            <scan>
-                <horizontal>
-                    <samples>360</samples>
-                    <resolution>1.0</resolution>
-                    <min_angle>-1.5708</min_angle>
-                    <max_angle>1.5708</max_angle>
-                </horizontal>
-            </scan>
-            <range>
-                <min>0.2</min>
-                <max>12.0</max>
-                <resolution>0.02</resolution>
-            </range>
-            <noise>
-                <type>gaussian</type>
-                <mean>0.0</mean>
-                <stddev>0.01</stddev>
-            </noise>
-        </ray>
+  <gazebo reference="laser">
+    <sensor name="lidar" type="gpu_lidar">
+      <always_on>true</always_on>
+      <visualize>true</visualize>
+      <topic>scan</topic>
+      <update_rate>5</update_rate>
+      <gz_frame_id>laser</gz_frame_id>
+      <lidar>
+        <scan>
+          <horizontal>
+            <samples>360</samples>
+            <resolution>1.00000</resolution>
+            <min_angle>0.000000</min_angle>
+            <max_angle>6.280000</max_angle>
+          </horizontal>
+        </scan>
+        <range>
+          <min>0.120000</min>
+          <max>12.0</max>
+          <resolution>0.02</resolution>
+        </range>
+        <noise>
+          <type>gaussian</type>
+          <mean>0.0</mean>
+          <stddev>0.01</stddev>
+        </noise>
+      </lidar>
     </sensor>
   </gazebo>

File: src/amiibot_description/urdf/amiibot_ros2_control.xacro (robot description, xacro)
@@ -1,38 +1,29 @@
 <?xml version="1.0"?>
 <robot name="amiibot" xmlns:xacro="http://www.ros.org/wiki/xacro">
-    <ros2_control name ="RobotSystem" type="system">
-    <!-- FOR SIMULATION, WITOUT REAL HARDWARE OR WITH ROBOCLAW
-      <hardware>
-        <plugin>mock_components/GenericSystem</plugin>
-        <param name="calculate_dynamics">true</param>
-        <plugin>roboclaw_hardware_interface/RoboClawHardwareInterface</plugin>
-          <param name="serial_port">/dev/ttyACM0</param>
-          <param name="serial_baud" type="int">115200</param>
-      </hardware>
-      <joint name="left_wheel_joint">
-        <command_interface name="velocity"/>
-        <state_interface name="position"/>
-        <param name="address">128</param>
-        <param name="motor_type">M2</param>
-        <param name="qppr">33800</param>
-      </joint>
-      <joint name="right_wheel_joint">
-        <command_interface name="velocity"/>
-        <state_interface name="position"/>
-        <param name="address">128</param>
-        <param name="motor_type">M1</param>
-        <param name="qppr">33800</param>
-      </joint>
-      -->
-      <hardware>
-          <plugin>odrive_ros2_control_plugin/ODriveHardwareInterface</plugin>
-          <param name="can">can1</param>
-      </hardware>
-      <joint name="left_wheel_joint">
-        <param name="node_id">0</param>
-      </joint>
-      <joint name="right_wheel_joint">
-        <param name="node_id">1</param>
-      </joint>
+    <ros2_control name="RobotSystem" type="system">
+        <!-- SIMULATION: Gazebo System Interface -->
+        <xacro:if value="$(arg is_simulation)">
+            <hardware>
+                <plugin>ign_ros2_control/IgnitionSystem</plugin>
+            </hardware>
+        </xacro:if>
+        <!-- REAL HARDWARE: ODrive motor controller -->
+        <xacro:unless value="$(arg is_simulation)">
+            <hardware>
+                <plugin>odrive_ros2_control_plugin/ODriveHardwareInterface</plugin>
+                <param name="can">can1</param>
+            </hardware>
+        </xacro:unless>
+        <!-- Joint interfaces (common for both sim and real) -->
+        <joint name="left_wheel_joint">
+            <command_interface name="velocity"/>
+            <state_interface name="position"/>
+            <state_interface name="velocity"/>
+        </joint>
+        <joint name="right_wheel_joint">
+            <command_interface name="velocity"/>
+            <state_interface name="position"/>
+            <state_interface name="velocity"/>
+        </joint>
     </ros2_control>
 </robot>
