Commit message: Refactor Isaac URDF: standalone xacro with find-resolved mesh paths, box collision on base_link

File: src/amiibot_description/urdf/amiibot_isaac.urdf.xacro (robot description, xacro)
@@ -1,13 +1,233 @@
 <?xml version="1.0"?>
 <!--
-  URDF for Isaac Sim 5.1.0
-  - Includes only robot geometry (amiibot_base.xacro)
-  - No Gazebo/Ignition plugins
-  - No ros2_control block (differential drive is configured via OmniGraph in Isaac Sim)
-  To export a resolved URDF (recommended before importing into Isaac Sim):
+  URDF for Isaac Sim 5.1.0 — standalone, no Gazebo plugins, no ros2_control.
+  Mesh paths use $(find ...) so xacro resolves them to absolute paths on export.
+  amiibot_base.xacro stays untouched (uses package:// for Ignition).
+  To export:
     source install/setup.bash
-    xacro src/amiibot_description/urdf/amiibot_isaac.urdf.xacro > /tmp/amiibot_isaac.urdf
+    bash scripts/export_isaac_urdf.sh
 -->
 <robot name="amiibot" xmlns:xacro="http://www.ros.org/wiki/xacro">
-    <xacro:include filename="$(find amiibot_description)/urdf/amiibot_base.xacro"/>
+    <xacro:property name="mesh_path" value="$(find amiibot_description)/meshes"/>
+    <!-- LINKS -->
+    <link name="base_footprint"/>
+    <link name="base_link">
+        <visual>
+            <origin xyz="0 0 0" rpy="1.5708 0 1.5708"/>
+            <geometry>
+                <mesh filename="${mesh_path}/base_link_300.stl" scale="0.001 0.001 0.001"/>
+            </geometry>
+            <material name="white">
+                <color rgba="1.0 1.0 1.0 1.0"/>
+            </material>
+        </visual>
+        <collision>
+            <origin xyz="0 0 0" rpy="0 0 0"/>
+            <geometry>
+                <box size="0.45 0.35 0.28"/>
+            </geometry>
+        </collision>
+        <inertial>
+            <origin xyz="0 0 0" rpy="0 0 0"/>
+            <mass value="30.0"/>
+            <inertia
+              ixx="0.637399" ixy="-0.005718" ixz="0.005136"
+              iyy="1.043697" iyz="0.010418"
+              izz="0.711315"/>
+        </inertial>
+    </link>
+    <link name="left_wheel">
+        <visual>
+            <origin xyz="0 0 0" rpy="1.5708 0 0"/>
+            <geometry>
+                <cylinder radius="0.0855" length="0.04"/>
+            </geometry>
+            <material name="black">
+                <color rgba="0.0 0.0 0.0 1.0"/>
+            </material>
+        </visual>
+        <collision>
+            <origin xyz="0 0 0" rpy="1.5708 0 0"/>
+            <geometry>
+                <cylinder radius="0.0855" length="0.04"/>
+            </geometry>
+        </collision>
+        <inertial>
+            <origin xyz="0 0 0" rpy="0 0 0"/>
+            <mass value="1.0"/>
+            <inertia
+              ixx="0.0116" ixy="0" ixz="0"
+              iyy="0.0063" iyz="0"
+              izz="0.0063"/>
+        </inertial>
+    </link>
+    <link name="right_wheel">
+        <visual>
+            <origin xyz="0 0 0" rpy="1.5708 0 0"/>
+            <geometry>
+                <cylinder radius="0.0855" length="0.04"/>
+            </geometry>
+            <material name="black">
+                <color rgba="0.0 0.0 0.0 1.0"/>
+            </material>
+        </visual>
+        <collision>
+            <origin xyz="0 0 0" rpy="1.5708 0 0"/>
+            <geometry>
+                <cylinder radius="0.0855" length="0.04"/>
+            </geometry>
+        </collision>
+        <inertial>
+            <origin xyz="0 0 0" rpy="0 0 0"/>
+            <mass value="1.0"/>
+            <inertia
+              ixx="0.0116" ixy="0" ixz="0"
+              iyy="0.0063" iyz="0"
+              izz="0.0063"/>
+        </inertial>
+    </link>
+    <link name="front_caster_wheel">
+        <visual>
+            <origin xyz="0 0 0" rpy="0 0 0"/>
+            <geometry>
+                <sphere radius="0.04"/>
+            </geometry>
+            <material name="gray">
+                <color rgba="0.6 0.6 0.6 1.0"/>
+            </material>
+        </visual>
+        <collision>
+            <origin xyz="0 0 0" rpy="0 0 0"/>
+            <geometry>
+                <sphere radius="0.04"/>
+            </geometry>
+        </collision>
+        <inertial>
+            <origin xyz="0 0 0" rpy="0 0 0"/>
+            <mass value="0.2"/>
+            <inertia ixx="0.01" ixy="0" ixz="0" iyy="0.01" iyz="0" izz="0.01"/>
+        </inertial>
+    </link>
+    <link name="back_caster_wheel">
+        <visual>
+            <origin xyz="0 0 0" rpy="0 0 0"/>
+            <geometry>
+                <sphere radius="0.04"/>
+            </geometry>
+            <material name="gray">
+                <color rgba="0.6 0.6 0.6 1.0"/>
+            </material>
+        </visual>
+        <collision>
+            <origin xyz="0 0 0" rpy="0 0 0"/>
+            <geometry>
+                <sphere radius="0.04"/>
+            </geometry>
+        </collision>
+        <inertial>
+            <origin xyz="0 0 0" rpy="0 0 0"/>
+            <mass value="0.2"/>
+            <inertia ixx="0.01" ixy="0" ixz="0" iyy="0.01" iyz="0" izz="0.01"/>
+        </inertial>
+    </link>
+    <link name="imu">
+        <visual>
+            <origin xyz="0 0 0" rpy="0 0 0"/>
+            <geometry>
+                <box size="0.03 0.03 0.01"/>
+            </geometry>
+            <material name="gray">
+                <color rgba="0.3 0.3 0.3 1"/>
+            </material>
+        </visual>
+    </link>
+    <link name="laser">
+        <visual>
+            <origin xyz="0 0 -0.025" rpy="1.5708 0 -1.5708"/>
+            <geometry>
+                <mesh filename="${mesh_path}/lidar.stl" scale="0.001 0.001 0.001"/>
+            </geometry>
+            <material name="black">
+                <color rgba="0.1 0.1 0.1 1"/>
+            </material>
+        </visual>
+    </link>
+    <link name="microphone">
+        <visual>
+            <origin xyz="0 0 0" rpy="0 0 0"/>
+            <geometry>
+                <cylinder radius="0.1" length="0.02"/>
+            </geometry>
+            <material name="gray">
+                <color rgba="0.3 0.3 0.3 1"/>
+            </material>
+        </visual>
+    </link>
+    <link name="depth_camera">
+        <visual>
+            <origin xyz="0 0 0" rpy="0 0 0"/>
+            <geometry>
+                <box size="0.025 0.1 0.03"/>
+            </geometry>
+            <material name="gray">
+                <color rgba="0.3 0.3 0.3 1"/>
+            </material>
+        </visual>
+    </link>
+    <!-- JOINTS -->
+    <joint name="base_joint" type="fixed">
+        <parent link="base_footprint"/>
+        <child link="base_link"/>
+        <origin xyz="0 0 0.04" rpy="0 0 0"/>
+    </joint>
+    <joint name="left_wheel_joint" type="continuous">
+        <parent link="base_link"/>
+        <child link="left_wheel"/>
+        <origin xyz="0 0.1725 0.0455" rpy="0 0 0"/>
+        <axis xyz="0 -1 0"/>
+        <dynamics damping="0.2"/>
+    </joint>
+    <joint name="right_wheel_joint" type="continuous">
+        <parent link="base_link"/>
+        <child link="right_wheel"/>
+        <origin xyz="0 -0.1725 0.0455" rpy="0 0 0"/>
+        <axis xyz="0 1 0"/>
+        <dynamics damping="0.2"/>
+    </joint>
+    <joint name="front_caster_joint" type="fixed">
+        <origin xyz="0.2075 0 0" rpy="0 0 0"/>
+        <parent link="base_link"/>
+        <child link="front_caster_wheel"/>
+    </joint>
+    <joint name="back_caster_joint" type="fixed">
+        <origin xyz="-0.2075 0 0" rpy="0 0 0"/>
+        <parent link="base_link"/>
+        <child link="back_caster_wheel"/>
+    </joint>
+    <joint name="imu_joint" type="fixed">
+        <parent link="base_link"/>
+        <child link="imu"/>
+        <origin xyz="0 0 0.10" rpy="0 0 0"/>
+    </joint>
+    <joint name="laser_joint" type="fixed">
+        <parent link="base_link"/>
+        <child link="laser"/>
+        <origin xyz="0.16 0 0.325" rpy="0 0 3.14159265"/>
+    </joint>
+    <joint name="microphone_joint" type="fixed">
+        <parent link="base_link"/>
+        <child link="microphone"/>
+        <origin xyz="0 0 1.2" rpy="0 0 0"/>
+    </joint>
+    <joint name="depth_camera_joint" type="fixed">
+        <parent link="base_link"/>
+        <child link="depth_camera"/>
+        <origin xyz="0.14 0 0.6" rpy="0 0 0"/>
+    </joint>
+    <link name="depth_camera_optical_frame"/>
+    <joint name="depth_camera_optical_joint" type="fixed">
+        <parent link="depth_camera"/>
+        <child link="depth_camera_optical_frame"/>
+        <origin xyz="0 0 0" rpy="0 0 0"/>
+    </joint>
 </robot>

File: src/amiibot_description/urdf/isaac/amiibot_isaac.urdf (robot description, URDF)
Before this commit: robot amiibot, 11 links, 10 joints
Links:
- link base_link: geometry collision box size=0.45 0.35 0.28; visual mesh filename=/home/gr/amiibot_ws/install/amiibot_description/share/amiib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 scale=0.001 0.001 0.001
Joints:
- joint back_caster_joint: axis 0 0 0 -> (none)
- joint front_caster_joint: axis 0 0 0 -> (none)
