Commit message: Add Nav2 support: fix costmap, EKF, SLAM map and navigation launch
- Fix twist_mux output topic to cmd_vel_unstamped (matches diff_drive_controller)
- Set imu0_differential: true in EKF to avoid yaw oscillation near +-180 deg
- Fix nav2_params: correct bt_navigator plugin name (nav2_round_robin_node_bt_node)
- Make map file a launch argument in nav2_bringup.launch.py (default: small_house_map)
- Add small_house_map (pgm + yaml) generated via SLAM toolbox
- Add slam_display.rviz config for SLAM sessions

Co-Authored-By: Claude Sonnet 4.6 <noreply@anthropic.com>

File: src/amiibot_description/urdf/amiibot_base.xacro (robot description, xacro)
@@ -190,5 +190,5 @@
       <parent link="base_link"/>
       <child link="imu"/>
-      <origin xyz="0 0 0.28" rpy="0 0 0"/>
+      <origin xyz="0 0 0.10" rpy="0 0 0"/>
     </joint>
     <joint name="laser_joint" type="fixed">

Commit message: Add RealSense D435 depth camera: URDF, Gazebo plugin, scan_depth for Nav2
- Add depth_camera link (box) + optical frame to URDF
- Add rgbd_camera sensor plugin in amiibot_gazebo.xacro (D435 specs: 87deg FOV, 0.3-10m)
- Add depth camera bridge topics to gazebo.launch.py (image, depth_image, points, camera_info)
- Replace depthimage_to_laserscan with pointcloud_to_laserscan (avoids optical frame issues)
- Add /scan_depth as second observation source in Nav2 local costmap voxel_layer

Co-Authored-By: Claude Sonnet 4.6 <noreply@anthropic.com>

File: src/amiibot_description/urdf/amiibot_base.xacro (robot description, xacro)
@@ -155,4 +155,15 @@
       </visual>
     </link>
+    <link name="depth_camera">
+      <visual>
+        <origin xyz="0 0 0" rpy="0 0 0"/>
+        <geometry>
+          <box size="0.025 0.1 0.03"/>
+        </geometry>
+        <material name="gray">
+          <color rgba="0.3 0.3 0.3 1"/>
+        </material>
+      </visual>
+    </link>
     <!-- JOINTS -->
     <joint name="base_joint" type="fixed">
@@ -202,3 +213,14 @@
       <origin xyz="0 0 1.2" rpy="0 0 0"/>
     </joint>
+    <joint name="depth_camera_joint" type="fixed">
+      <parent link="base_link"/>
+      <child link="depth_camera"/>
+      <origin xyz="0.12 0 0.6" rpy="0 0 0"/>
+    </joint>
+    <link name="depth_camera_optical_frame"/>
+    <joint name="depth_camera_optical_joint" type="fixed">
+      <parent link="depth_camera"/>
+      <child link="depth_camera_optical_frame"/>
+      <origin xyz="0 0 0" rpy="0 0 0"/>
+    </joint>
 </robot>

File: src/amiibot_description/urdf/amiibot_gazebo.xacro (robot description, xacro)
@@ -115,3 +115,23 @@
     </sensor>
   </gazebo>
+  <!-- Depth Camera (RealSense D435) -->
+  <gazebo reference="depth_camera">
+    <sensor name="depth_camera" type="rgbd_camera">
+      <always_on>true</always_on>
+      <update_rate>15</update_rate>
+      <topic>depth_camera</topic>
+      <gz_frame_id>depth_camera_optical_frame</gz_frame_id>
+      <camera>
+        <horizontal_fov>1.5184</horizontal_fov>
+        <image>
+          <width>640</width>
+          <height>480</height>
+        </image>
+        <clip>
+          <near>0.3</near>
+          <far>10.0</far>
+        </clip>
+      </camera>
+    </sensor>
+  </gazebo>
 </robot>

Commit message: Add Isaac Sim 5.1.0 full integration: URDF, Nav2, SLAM, sensors
- amiibot_isaac.launch.py: EKF, static TFs, pointcloud_to_laserscan,
  slam_toolbox (use_slam:=true) and Nav2 (use_slam:=false) modes
- nav2_params_isaac.yaml: BEST_EFFORT QoS for /scan, initial pose at
  origin, smoother_server and velocity_smoother config
- slam_params_isaac.yaml: slam_toolbox async mapping config
- ekf_isaac.yaml: EKF with use_sim_time for Isaac Sim
- nav2_bringup.launch.py: added params_file argument for per-sim config
- Isaac URDF/USD assets and scene file
- RViz configs for Isaac Sim and Nav2
- Maps: isaac_map (Simple Room) and bookstore_map

Co-Authored-By: Claude Sonnet 4.6 <noreply@anthropic.com>

File: src/amiibot_description/urdf/amiibot_base.xacro (robot description, xacro)
@@ -7,5 +7,5 @@
             <origin xyz="0 0 0" rpy="1.5708 0 1.5708"/>
             <geometry>
-                <mesh filename="package://amiibot_description/meshes/base_link.stl" scale="0.001 0.001 0.001"/>
+                <mesh filename="package://amiibot_description/meshes/base_link_300.stl" scale="0.001 0.001 0.001"/>
             </geometry>
             <material name="white">
@@ -206,5 +206,5 @@
       <parent link="base_link"/>
       <child link="laser"/>
-      <origin xyz="0.16 0 0.285" rpy="0 0 3.14159265"/>
+      <origin xyz="0.16 0 0.325" rpy="0 0 3.14159265"/>
     </joint>
     <joint name="microphone_joint" type="fixed">
@@ -216,5 +216,5 @@
       <parent link="base_link"/>
       <child link="depth_camera"/>
-      <origin xyz="0.12 0 0.6" rpy="0 0 0"/>
+      <origin xyz="0.14 0 0.6" rpy="0 0 0"/>
     </joint>
     <link name="depth_camera_optical_frame"/>

File: src/amiibot_description/urdf/amiibot_gazebo.xacro (robot description, xacro)
@@ -86,4 +86,10 @@
     </sensor>
   </gazebo>
+  <!-- base_link usa visibility_flags=1 para ser invisible al LiDAR (gpu_lidar filtra por mask) -->
+  <gazebo reference="base_link">
+    <visual>
+      <visibility_flags>1</visibility_flags>
+    </visual>
+  </gazebo>
   <gazebo reference="laser">
     <sensor name="lidar" type="gpu_lidar">
@@ -93,4 +99,5 @@
       <update_rate>5</update_rate>
       <gz_frame_id>laser</gz_frame_id>
+      <visibility_mask>4294967294</visibility_mask>
       <lidar>
         <scan>

File: src/amiibot_description/urdf/amiibot_isaac.urdf.xacro (robot description, xacro)
@@ -23,5 +23,5 @@
         </visual>
         <collision>
-            <origin xyz="0 0 0" rpy="0 0 0"/>
+            <origin xyz="0 0 0.20" rpy="0 0 0"/>
             <geometry>
                 <box size="0.45 0.35 0.28"/>
@@ -185,5 +185,5 @@
         <child link="left_wheel"/>
         <origin xyz="0 0.1725 0.0455" rpy="0 0 0"/>
-        <axis xyz="0 -1 0"/>
+        <axis xyz="0 1 0"/>
         <dynamics damping="0.2"/>
     </joint>

File: src/amiibot_description/urdf/isaac/amiibot_isaac.urdf (robot description, URDF)
Before this commit: robot amiibot, 11 links, 10 joints
Joints:
- joint left_wheel_joint: axis 0 -1 0 -> 0 1 0
